Commit message: Update roseco.gazebo.xacro

File: roseco_description/urdf/roseco.gazebo.xacro (robot description, xacro)
@@ -6,25 +6,24 @@
       <robotNamespace>/roseco</robotNamespace>
       <!--robotParam>/robot_description</robotParam-->
-      <robotSimType>gazebo_ros_control/DefaultRobotHWSim</robotSimType>
+      <!--<robotSimType>gazebo_ros_control/DefaultRobotHWSim</robotSimType>-->
+      <commandTopic>cmd_vel</commandTopic>
+      <odometryTopic>odom</odometryTopic>
+      <odometryFrame>odom</odometryFrame>
+      <odometrySource>world</odometrySource>
+      <publishOdomTF>true</publishOdomTF>
+      <robotBaseFrame>base_footprint</robotBaseFrame>
+      <publishWheelTF>false</publishWheelTF>
+      <publishTf>true</publishTf>
+      <publishWheelJointState>true</publishWheelJointState>
+      <legacyMode>false</legacyMode>
+      <updateRate>30</updateRate>
+      <leftJoint>wheel_left_joint</leftJoint>
+      <rightJoint>wheel_right_joint</rightJoint>
+      <wheelSeparation>0.15</wheelSeparation>
+      <wheelDiameter>0.17164</wheelDiameter>
+      <wheelAcceleration>1</wheelAcceleration>
+      <wheelTorque>10</wheelTorque>
+      <rosDebugLevel>na</rosDebugLevel>
     </plugin>
   </gazebo>
-  <!-- xacro to set the friction for the wheel. This patch was taken from the MIR
-  repository.
-    https://github.com/dfki-ric/mir_robot/tree/noetic.
-    https://github.com/dfki-ric/mir_robot/blob/a216d7374c21e360c94034d360b07fd7a4d42842/mir_description/urdf/include/mir_100.gazebo.xacro#L29
-   -->
-  <xacro:macro name="set_wheel_friction" params="link friction">
-    <gazebo reference="${link}">
-      <mu1 value="${friction}"/>
-      <mu2 value="${friction}"/>
-      <kp value="10000000.0"/>
-      <kd value="1.0"/>
-      <minDepth>0.01</minDepth>
-    </gazebo>
-  </xacro:macro>
-  <xacro:macro name="set_all_wheel_frictions" >
-    <xacro:set_wheel_friction link="left_wheel" friction="200"/>
-    <xacro:set_wheel_friction link="riht_wheel" friction="200"/>
-    <xacro:set_wheel_friction link="caster_wheel" friction="200"/>
-  </xacro:macro>
 </robot>
